Commit message: submission video capture point

File: src/robot/turtlebot3_description/urdf/turtlebot3_waffle.urdf.xacro (robot description, xacro)
@@ -25,5 +25,5 @@
             <origin xyz="-0.064 0 0.047" rpy="0 0 0"/>
             <geometry>
-                <box size="0.266 0.266 0.094"/>
+                <box size="0.1 0.1 0.094"/>
             </geometry>
         </collision>
